Commit message: table rough draft

File: data/table/table.urdf (robot description, URDF)
Before this commit: robot table.urdf, 1 links, 0 joints
Links:
- link baseLink: mass .0 -> 5; geometry collision box size=1.5 1 .9; visual mesh filename=table.obj scale=0.1 0.1 .92

Commit message: urdf changes

File: data/table/table.urdf (robot description, URDF)
Before this commit: robot table.urdf, 1 links, 0 joints
Links:
- link baseLink: geometry collision box size=1.5 1 .85; visual mesh filename=tablebody.stl scale=1 1 1
