Commit message: Added Pick Place Env Code for Scripted Policy Test

File: data/table/puck.urdf (robot description, URDF)
Before this commit: robot puck.urdf, 1 links, 0 joints
Links:
- link baseLink: mass .05 -> 0.75; geometry collision cylinder length=.04 radius=.02; visual cylinder length=.04 radius=.02
